File: source/foc.kicad_sch (KiCad schematic)
At the start: 32 parts, among them J1 Conn_01x02_Male, J2 Conn_01x06, J3 communication, SW1 SW_DPDT_x2, U1 TJA1051T/3/1J, U2 BMI160

Commit message: update IMU
Parts:
- added CAP1, CAP2: 100n, Capacitor_SMD:C_0603_1608Metric, symbol BLDC_4-rescue:C-RESCUE-BLDC_4
- added R3k: 3.3k, Resistor_SMD:R_0603_1608Metric, symbol BLDC_4-rescue:R-RESCUE-BLDC_4
- added R4k1: 4.02k, Resistor_SMD:R_0603_1608Metric, symbol BLDC_4-rescue:R-RESCUE-BLDC_4
- U2: value BMI160 -> ICM-20948; footprint Package_LGA:Bosch_LGA-14_3x2.5mm_P0.5mm -> Sensor_Motion:InvenSense_QFN-24_3x3mm_P0.4mm; symbol Cheap-FOCer-2-60mm-rescue:BMI160-IMU -> Sensor_Motion:ICM-20948
Connections:
- net GND: now also U2.18 (GND), U2.20 (GND), CAP1.1, CAP2.1, R4k1.2; no longer U2.1 (SDO), U2.6 (GNDIO), U2.7 (GND)
- net VCC: now also R3k.1; no longer U2.12 (CSB), U2.5 (VDDIO), U2.8 (VDD)
- net mcu/PB2: now also R7.2, U2.24 (SDA/SDI); no longer R6.1, U2.14 (SDX)
- net mcu/PA15: no longer names the net of U2.13 (VDD)
- net mcu/PA15: now also U2.8 (VDDIO), CAP1.2, CAP2.2, R3k.2, R4k1.1; no longer R7.2
- new net mcu/PB15: R6.1, U2.23 (SCL/SCLK)
- no-connect marks 17 -> 18
Other:
- sheet mcu ports: added PB15; removed PA15
- note added: "VDDIO (Voltage Divider to 1.812v)"
- moved on the sheet: C5, C6
